File: ports-GPIO.sch (KiCad schematic (older format))
At the start: 36 parts, among them J1 Conn_01x20_Male, J2 HDMI_A, J3 Conn_01x20_Male, J4 USB_B_Micro, Q1 MMBT3906, Q2 MMBT3906, Q3 MMBT3904, U8 SLS2301

Commit message: did some routing and fixed some pinouts on components
Parts:
- R32: footprint Resistor_SMD:R_0402_1005Metric -> (none)
Changed lines of the file:
@@
 U 1 1 5F6F6264
 P 9100 5200
+AR Path="/5F6F6264" Ref="J4"  Part="1"
+AR Path="/5F529CC2/5F6F6264" Ref="J4"  Part="1"
 F 0 "J4" H 9157 5667 50  0000 C CNN
 F 1 "USB_B_Micro" H 9157 5576 50  0000 C CNN
@@
 F 0 "R32" H 10680 2254 50  0000 R CNN
 F 1 "510R" H 10680 2345 50  0000 R CNN
-F 2 "Resistor_SMD:R_0402_1005Metric" V 10680 2300 50  0001 C CNN
+F 2 "" V 10680 2300 50  0001 C CNN
 F 3 "~" H 10750 2300 50  0001 C CNN
 	1    10750 2300
