File: card.sync-conflict-20210417-222047-TQHVD7P.kicad_pcb (KiCad board)
At the start: 2 copper layers, 38.6 x 52.3 mm, 83 parts, among them J1 Conn_01x20_Male, J2 HDMI_A, J3 Conn_01x20_Male, J4 USB_B_Micro, SW1 SW_DPST_x2, U1 SPX3819-1.8, U2 IMP811REUS-T, U3 SP6205EM5-L-3-3_TR, U4 MP1469GJ, U5 W25Q32JVSS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

Commit message: did more routing! allmost done now!
Parts:
- removed JP1, JP2: Jumper, Jumper:SolderJumper-2_P1.3mm_Open_TrianglePad1.0x1.5mm
- moved C13 0.30 mm to (244.1, 92.5)
- moved R6 0.30 mm to (242.8, 90.4)
- moved R9 0.30 mm to (242.8, 92.5)
Routing:
- net GND: track 344.2 -> 273.5 mm, vias 29 -> 13
- net +2V5: track 63.2 -> 3.29 mm, vias 2 -> 0
- net +1V8: track 53.0 -> 13.8 mm, vias 4 -> 0
- net +1V1: track 69.4 -> 33.8 mm, vias 4 -> 0
- net +5V: track 145.0 -> 119.1 mm, vias 5 -> 3
- net Net-(U7-Pad3): track 24.5 -> 0.00 mm, vias 2 -> 0
- net Net-(U7-Pad4): track 24.3 -> 0.00 mm, vias 2 -> 0
- net +3V3: track 206.9 -> 182.8 mm, vias 15 -> 13
- net TX2_P: track 25.9 -> 11.0 mm, vias 2 -> 1
- net HOST1_DP: track 38.1 -> 34.2 mm, vias 3 -> 2
- net Net-(C12-Pad2): track 7.83 -> 4.62 mm
- net HOST0_DP: track 47.7 -> 50.6 mm
- net /CPU/SPI_CLK: track 14.8 -> 12.4 mm
- net HOST1_DM: track 33.4 -> 32.0 mm
- net VOUT1: track 33.6 -> 32.3 mm, vias 4 -> 2
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- removed copper zone on B.Cu, net GND
Other:
- board text removed: "solder for bluetooth"
